Commit message: added sonar plugin

File: FINAL/src/final_description/urdf/final.urdf (robot description, URDF)
Before this commit: robot final_description, 14 links, 13 joints
Links:
- added link sonar_link, mass 1e-5; collision box size=0.01 0.01 0.01; visual box size=0.01 0.01 0.01
Joints:
- added joint sonar_front_joint: type fixed, parent LA, child sonar_link, origin xyz=0.13 0.015 -0.02 rpy=3.1415926 0 -1.570796326, axis 0 1 0
