Commit message: Add files via upload
With all the essentials, SONAR included...FINAL

File: FINAL/Mechanical/bot1/urdf/bot1.urdf (robot description, URDF)
Before this commit: robot bot1, 15 links, 14 joints
Links:
- removed link LC
- removed link RC
- added link hokuyo_link, mass 1e-5; collision box size=0.1 0.1 0.1; visual mesh filename=package://bot1/meshes/hokuyo.dae
- added link sonar_link, mass 1e-5; collision box size=0.01 0.01 0.01; visual box size=0.01 0.01 0.01
- link LF: mass 0.24614 -> 0.35
- link RF: mass 0.24614 -> 0.30
- link base_link: geometry collision mesh filename=package://bot1/meshes/base_link.STL scale=1 1 1; visual mesh filename=package://bot1/meshes/base_link.STL
Joints:
- removed joint LCJ
- removed joint RCJ
- added joint hokuyo_joint: type fixed, parent F, child hokuyo_link, origin xyz=0.04 0.05 0 rpy=-1.57 0 0, axis 0 1 0
- added joint sonar_front_joint: type fixed, parent LA, child sonar_link, origin xyz=0.13 0.015 -0.02 rpy=3.1415926 0 -1.570796326, axis 0 1 0
- joint BJ: limit lower=-0.15 upper=0 effort=100 velocity=0.1 -> lower=-0.15 upper=0 effort=1000 velocity=0.1
- joint FCJ: origin xyz=0.01 0.275 0 rpy=0 0 0 -> xyz=0.01 0.275 0 rpy=-1.57 0 0
- joint FJ: limit lower=-0.18 upper=0 effort=100 velocity=0.1 -> lower=-0.18 upper=0 effort=10 velocity=0.05
- joint LFJ: limit lower=-0.34 upper=1.36 effort=100 velocity=0.125 -> lower=-0.34 upper=1.36 effort=100 velocity=0.3; mimic (none) -> joint=RFJ multiplier=-1 offset=0
- joint RFJ: limit lower=-1.5 upper=0.2 effort=100 velocity=0.125 -> lower=-1.5 upper=0.2 effort=100 velocity=0.3
